File: hardware/t9kb.kicad_pcb (KiCad board)
At the start: 2 copper layers, 48 x 68 mm, 34 parts, among them J1 Qwiic, J2 Breakout, SW1 SOFT_L, SW10 CALL, SW11 DOWN, SW12 END, SW13 K1, SW14 K2, SW15 K3, SW16 K4, SW17 K5, SW18 K6, SW19 K7, SW2 SOFT_M, SW20 K8, SW21 K9, SW22 KSTAR, SW23 K0, SW24 KHASH, SW3 SOFT_R, SW4 SPK, SW5 UP, SW6 CONTACT, SW7 LEFT, SW8 OK, SW9 RIGHT, U1 TCA8418RTWR

Commit message: pcb v0.3: updated layout, gerbers and step
Parts:
- added H1: M1.4, MountingHole_1.5mm_M1.4, F.Cu at (146.8, 166.3)
- added H2: M1.4, MountingHole_1.5mm_M1.4, F.Cu at (101.4, 166.6)
- added H3: M1.4, MountingHole_1.5mm_M1.4, F.Cu at (146.7, 101.5)
- added H4: M1.4, MountingHole_1.5mm_M1.4, F.Cu at (101.5, 101.3)
Other:
- board text added: "T9KB v0.3 acidvegas"
- board text removed: "T9KB v0.2 acidvegas"
